File: corne-cherry/pcb_wl/v2/corne-cherry.sch (KiCad schematic (older format))
At the start: 72 parts, among them J1 MJ-4PP-9, J2 OLED, J3 Conn_01x02_Female, SW1 SW_PUSH, SW10 SW_PUSH, SW11 SW_PUSH, SW12 SW_PUSH, SW13 SW_PUSH, SW14 SW_PUSH, SW15 SW_PUSH, SW16 SW_PUSH, SW17 SW_PUSH, SW18 SW_PUSH, SW19 SW_PUSH, SW2 SW_PUSH, SW20 SW_PUSH, SW21 SW_PUSH, SW22 SW_PUSH, SW23 SW_SPDT, SW24 SW_SPDT, SW3 SW_PUSH, SW4 SW_PUSH, SW5 SW_PUSH, SW6 SW_PUSH, SW7 SW_PUSH, SW8 SW_PUSH, SW9 SW_PUSH, U1 ProMicro

Commit message: Bigger battery header, cleaner switch footprints and schematic
Parts:
- D1, D10, D11, D12, D13, D14, D15, D16, D17, D18, D19, D2, D20, D21, D3, D4, D5, D6, D7, D8, D9: footprint kbd:D3_TH_SMD -> kbd:D3_SMD
- G1, G2: footprint kbd:corne -> Silks:sporne-logo-small
- J1: symbol corne-cherry-rescue:MJ-4PP-9-kbd-corne-cherry-rescue -> kbd:MJ-4PP-9
- J3: footprint Connector_PinHeader_2.00mm:PinHeader_1x02_P2.00mm_Vertical -> kbd:Battery_Header
- RSW1: symbol corne-cherry-rescue:SW_PUSH-kbd-corne-cherry-rescue -> kbd:SW_PUSH
- SW1, SW10, SW11, SW12, SW13, SW14, SW15, SW16, SW17, SW18, SW19, SW2, SW20, SW3, SW4, SW5, SW6, SW7, SW8, SW9: footprint kbd:MX_ALPS_PG1350_noLed -> kbd:MX_Hitek_725_1U_reversible; symbol corne-cherry-rescue:SW_PUSH-kbd-corne-cherry-rescue -> kbd:SW_PUSH
- SW21: footprint kbd:CherryMX_MidHeight_Hotswap -> kbd:MX_Hitek_725_1.5U_reversible; symbol corne-cherry-rescue:SW_PUSH-kbd-corne-cherry-rescue -> kbd:SW_PUSH
- SW22: footprint kbd:CherryMX_MidHeight_Hotswap -> kbd:MX_Hitek_725_1U_reversible; symbol corne-cherry-rescue:SW_PUSH-kbd-corne-cherry-rescue -> kbd:SW_PUSH
- U1: symbol corne-cherry-rescue:ProMicro-kbd-corne-cherry-rescue -> kbd:ProMicro
Connections:
- net col0: no longer SW1.1, SW13.1, SW7.1
- net col1: no longer SW2.1, SW8.1
- net col2: no longer SW3.1, SW9.1
- net col3: no longer SW10.1, SW16.1, SW4.1
- net col4: no longer SW11.1, SW17.1, SW5.1
- net col5: no longer SW12.1, SW18.1, SW6.1
