File: corne-cherry/pcb_top/corne-top-plate-breakoff.kicad_pcb (KiCad board)
At the start: 2 copper layers, 151.9 x 91.4 mm, 27 parts, among them SW2 KEY_SWITCH

Commit message: Minor fixes, updated gerbers
Parts:
- SW2 (x22): footprint kbd:SW_Hole -> kbd:SW_Hole_ALPS
- turned SW2 to 60 degrees
